File: board/sio2sd.sch (KiCad schematic (older format))
At the start: 20 parts, among them CON1 SD_Card, IC1 ATMEGA328PB-A, P1 ICSP, P2 SIO, SW1 UP, SW2 DOWN, SW3 RESET

Commit message: Single board device design
Parts:
- removed P1: ICSP, Pin_Headers:Pin_Header_Angled_1x04_Pitch2.54mm, symbol CONN_01X04
- removed R1: 10k, Resistors_SMD:R_0805_HandSoldering, symbol R
- removed SW3: RESET, Buttons_Switches_SMD:SW_SPST_B3S-1000, symbol SW_PUSH
- added Q1: BC818-40, TO_SOT_Packages_SMD:SOT-23, symbol BC818-40
- added R1, R10: 10k, Resistors_SMD:R_0805_HandSoldering, symbol R_Small
- added W1: MOSI, footprints:pad, symbol TEST_1P
- added W2: MISO, footprints:pad, symbol TEST_1P
- added W3: SCK, footprints:pad, symbol TEST_1P
- added W4: Reset, footprints:pad, symbol TEST_1P
- CON1: footprint Connect:SD_Card_Receptacle -> footprints:sdcardsocket
- LED1: footprint (none) -> footprints:led2digit
- SW1, SW2: footprint Buttons_Switches_SMD:SW_SPST_B3S-1000 -> footprints:button
Connections:
- wire segments 109 -> 116
- no-connect marks 13 -> 9
Other:
- moved on the sheet: CON1

Commit message: Change reset circuit, layout fixes
Parts:
- removed Q1: BC818-40, TO_SOT_Packages_SMD:SOT-23, symbol BC818-40
- added C3: 100nF, Capacitors_SMD:C_0603_HandSoldering, symbol C_Small
- R1: value 10k -> 220k
Connections:
- wire segments 116 -> 115
Other:
- moved on the sheet: R10
Changed lines of the file:
@@
 encoding utf-8
 Sheet 1 1
-Title ""
+Title "SIO2SD single board"
 Date ""
-Rev ""
+Rev "1"
 Comp ""
 Comment1 ""
@@
 P 9800 4150
 F 0 "R1" H 9830 4170 50  0000 L CNN
-F 1 "10k" H 9830 4110 50  0000 L CNN
+F 1 "220k" H 9830 4110 50  0000 L CNN
 F 2 "Resistors_SMD:R_0805_HandSoldering" H 9800 4150 50  0001 C CNN
 F 3 "" H 9800 4150 50  0000 C CNN
@@
 Wire Wire Line
 	9800 4250 9800 5100
-Wire Wire Line
-	9800 4300 9950 4300
-Connection ~ 9800 4300
-Wire Wire Line
-	9800 3700 9800 4050
-$Comp
-L GND #PWR016
-U 1 1 5ACBD122
-P 10250 4600
-F 0 "#PWR016" H 10250 4350 50  0001 C CNN
-F 1 "GND" H 10250 4450 50  0000 C CNN
-F 2 "" H 10250 4600 50  0000 C CNN
-F 3 "" H 10250 4600 50  0000 C CNN
-	1    10250 4600
-	1    0    0    -1
-$EndComp
-Wire Wire Line
-	10250 4600 10250 4500
 $Comp
 L R_Small R10
 U 1 1 5ACBDB2D
-P 10250 3900
-F 0 "R10" H 10280 3920 50  0000 L CNN
-F 1 "10k" H 10280 3860 50  0000 L CNN
-F 2 "Resistors_SMD:R_0805_HandSoldering" H 10250 3900 50  0001 C CNN
-F 3 "" H 10250 3900 50  0000 C CNN
-	1    10250 3900
-	1    0    0    -1
-$EndComp
-Wire Wire Line
-	10250 4100 10250 4000
-$Comp
-L +3.3V #PWR017
+P 9800 3550
+F 0 "R10" H 9830 3570 50  0000 L CNN
+F 1 "10k" H 9830 3510 50  0000 L CNN
+F 2 "Resistors_SMD:R_0805_HandSoldering" H 9800 3550 50  0001 C CNN
+F 3 "" H 9800 3550 50  0000 C CNN
+	1    9800 3550
+	1    0    0    -1
+$EndComp
+Wire Wire Line
+	9800 3650 9800 4050
+$Comp
+L +3.3V #PWR016
 U 1 1 5ACBE4CA
-P 10250 3600
-F 0 "#PWR017" H 10250 3450 50  0001 C CNN
-F 1 "+3.3V" H 10250 3740 50  0000 C CNN
-F 2 "" H 10250 3600 50  0000 C CNN
-F 3 "" H 10250 3600 50  0000 C CNN
-	1    10250 3600
-	1    0    0    -1
-$EndComp
-Wire Wire Line
-	10250 3600 10250 3800
-Wire Wire Line
-	9800 3700 10250 3700
-Connection ~ 10250 3700
-Text Label 10550 4050 0    60   ~ 0
+P 9800 3250
+F 0 "#PWR016" H 9800 3100 50  0001 C CNN
+F 1 "+3.3V" H 9800 3390 50  0000 C CNN
+F 2 "" H 9800 3250 50  0000 C CNN
+F 3 "" H 9800 3250 50  0000 C CNN
+	1    9800 3250
+	1    0    0    -1
+$EndComp
+Wire Wire Line
+	9800 3250 9800 3450
+Text Label 9200 3900 0    60   ~ 0
 Reset
 $Comp
@@
 	5600 7100 5600 7000
 Wire Wire Line
-	10550 4050 10250 4050
-Connection ~ 10250 4050
-$Comp
-L BC818-40 Q1
-U 1 1 5ACC2DCA
-P 10150 4300
-F 0 "Q1" H 10350 4375 50  0000 L CNN
-F 1 "BC818-40" H 10350 4300 50  0000 L CNN
-F 2 "TO_SOT_Packages_SMD:SOT-23" H 10350 4225 50  0000 L CIN
-F 3 "" H 10150 4300 50  0000 L CNN
-	1    10150 4300
-	1    0    0    -1
-$EndComp
-Wire Wire Line
 	9800 5200 9950 5200
 Connection ~ 9950 5400
+$Comp
+L C_Small C3
+U 1 1 5AD32337
+P 10050 4150
+F 0 "C3" H 10060 4220 50  0000 L CNN
+F 1 "100nF" H 10060 4070 50  0000 L CNN
+F 2 "Capacitors_SMD:C_0603_HandSoldering" H 10050 4150 50  0001 C CNN
+F 3 "" H 10050 4150 50  0000 C CNN
+	1    10050 4150
+	1    0    0    -1
+$EndComp
+Wire Wire Line
+	9200 3900 10050 3900
+Wire Wire Line
+	10050 3900 10050 4050
+Connection ~ 9800 3900
+Wire Wire Line
+	10050 4250 10050 4400
+Wire Wire Line
+	10050 4400 9800 4400
+Connection ~ 9800 4400
 $EndSCHEMATC

Commit message: Allow multi-slave configuration
By inserting a diode into TX -> Data In, the device can emulate an open
collector to not interfer with other devices on the same bus.
Parts:
- added D1: 0.2V, Diodes_SMD:D_MicroMELF_Hadsoldering, symbol D_Schottky_Small
Connections:
- net TX: now also D1.2 (A); no longer IC1.31 ((TXD0/OC4A/PTCXY)PD1)
- new net: D1.1 (K), IC1.31 ((TXD0/OC4A/PTCXY)PD1)
Changed lines of the file:
@@
 Title "SIO2SD single board"
 Date ""
-Rev "1"
+Rev "2"
 Comp ""
 Comment1 ""
@@
 Text Label 6400 3600 0    60   ~ 0
 RX
-Text Label 6400 3500 0    60   ~ 0
-TX
 Text Label 6400 3700 0    60   ~ 0
 CMD
@@
 	4800 3600 6750 3600
 Wire Wire Line
-	5700 3500 6750 3500
-Wire Wire Line
-	5700 3500 5700 3700
-Wire Wire Line
-	5700 3700 4800 3700
-Wire Wire Line
 	3400 1250 3400 1600
 Wire Wire Line
@@
 	10050 4400 9800 4400
 Connection ~ 9800 4400
+$Comp
+L D_Schottky_Small D1
+U 1 1 5ADC4B95
+P 6100 3500
+F 0 "D1" H 6050 3580 50  0000 L CNN
+F 1 "0.2V" H 5900 3550 50  0000 C CNN
+F 2 "Diodes_SMD:D_MicroMELF_Hadsoldering" V 6100 3500 50  0001 C CNN
+F 3 "" V 6100 3500 50  0000 C CNN
+	1    6100 3500
+	1    0    0    -1
+$EndComp
+Text Label 6400 3500 0    60   ~ 0
+TX
+Wire Wire Line
+	5700 3700 4800 3700
+Wire Wire Line
+	5700 3500 5700 3700
+Wire Wire Line
+	5700 3500 6000 3500
+Wire Wire Line
+	6200 3500 6750 3500
 $EndSCHEMATC

Commit message: Bring design files to new KiCAD version. Create gerber files.
Parts:
- C1: footprint Capacitors_SMD:C_0805_HandSoldering -> Capacitor_SMD:C_0805_2012Metric_Pad1.15x1.40mm_HandSolder; symbol C_Small -> Device:C_Small
- C2, C3: footprint Capacitors_SMD:C_0603_HandSoldering -> Capacitor_SMD:C_0603_1608Metric_Pad1.05x0.95mm_HandSolder; symbol C_Small -> Device:C_Small
- CON1: symbol SD_Card -> sio2sd-rescue:SD_Card
- D1: footprint Diodes_SMD:D_MicroMELF_Hadsoldering -> Diode_SMD:D_0805_2012Metric_Pad1.15x1.40mm_HandSolder; symbol D_Schottky_Small -> Device:D_Schottky_Small
- IC1: footprint Housings_QFP:TQFP-32_7x7mm_Pitch0.8mm -> Package_QFP:TQFP-32_7x7mm_P0.8mm; symbol ATMEGA328PB-A -> sio2sd-rescue:ATMEGA328PB-A
- LED1: symbol LED2DIGIT -> components:LED2DIGIT
- P2: footprint Pin_Headers:Pin_Header_Angled_1x05_Pitch2.54mm -> Connector_PinHeader_2.54mm:PinHeader_1x05_P2.54mm_Horizontal; symbol CONN_01X05 -> sio2sd-rescue:CONN_01X05
- R1, R10: footprint Resistors_SMD:R_0805_HandSoldering -> Resistor_SMD:R_0805_2012Metric_Pad1.15x1.40mm_HandSolder; symbol R_Small -> Device:R_Small
- R2, R3, R4, R5, R6, R7, R8, R9: footprint Resistors_SMD:R_0805_HandSoldering -> Resistor_SMD:R_0805_2012Metric_Pad1.15x1.40mm_HandSolder; symbol R -> Device:R
- REG1: footprint TO_SOT_Packages_SMD:SOT-223 -> Package_TO_SOT_SMD:SOT-223; symbol LM1117IMPX-3.3 -> components:LM1117IMPX-3.3
- SW1, SW2: symbol SW_PUSH -> sio2sd-rescue:SW_PUSH
- W1, W2, W3, W4: symbol TEST_1P -> sio2sd-rescue:TEST_1P
